File: hardware/PCB/v0.2/PowerAndCommModule.kicad_sch (KiCad schematic)
At the start: 18 parts, among them J1 Screw_Terminal_01x02, J2 Conn_01x06_Pin, J3 Screw_Terminal_01x02, J4 Conn_01x04_Socket, J5 Screw_Terminal_01x02, K1 HF49FD_005-1H22G, Q1 S8050, SW1 SW_DIP_x01, U1 AMS1117-3.3, U2 ESP-32s

Commit message: commit before system update
Parts:
- C1: footprint Capacitor_Tantalum_SMD:CP_EIA-3216-18_Kemet-A_Pad1.58x1.35mm_HandSolder -> Capacitor_Tantalum_SMD:CP_EIA-3528-21_Kemet-B_Pad1.50x2.35mm_HandSolder
- J2: footprint Connector_PinHeader_2.00mm:PinHeader_1x06_P2.00mm_Vertical -> Connector_PinHeader_2.54mm:PinHeader_1x06_P2.54mm_Vertical
- J4: value Conn_01x04_Socket -> Conn_01x05_Socket
- K1: value HF49FD_005-1H22G -> HF49FD_005-1H11G; footprint HF49FD_005:HF49FD0051H22G -> HF49FD_005-1H11:HF49FD0051H11F
- SW1: footprint Button_Switch_THT:SW_PUSH_6mm_H4.3mm -> Button_Switch_SMD:SW_SPST_CK_RS282G05A3
Connections:
- net LINE: now also J1.2 (Pin_2), K1.2 (NO); no longer J1.1 (Pin_1), K1.1 (COM)
- net LINE_NO: now also J5.1 (Pin_1), K1.1 (COM); no longer J5.2 (Pin_2), K1.2 (NO)
- net NEUT: now also J1.1 (Pin_1), J5.2 (Pin_2); no longer J1.2 (Pin_2), J5.1 (Pin_1)
- net at SW1.1: now also U2.36 (IO22); no longer U2.16 (IO13)
Other:
- moved on the sheet: J1, J4, J5, R3, R4, SW1
